Commit message: update completed source

File: src/usv_description/urdf/gazebo.xacro (robot description, xacro)
@@ -46,8 +46,11 @@
           </horizontal>
           <vertical>
-            <samples>16</samples>
+            <!-- slam_toolbox consumes a 2D LaserScan. Keep one horizontal
+                 layer; ros_gz_bridge otherwise exposes the downward-most
+                 layer, which measures the water/pond surface at about 2.6 m. -->
+            <samples>1</samples>
             <resolution>1</resolution>
-            <min_angle>-0.741765</min_angle>
-            <max_angle>0.392699</max_angle>
+            <min_angle>0.0</min_angle>
+            <max_angle>0.0</max_angle>
           </vertical>
         </scan>
@@ -75,8 +78,8 @@
           </horizontal>
           <vertical>
-            <samples>16</samples>
+            <samples>1</samples>
             <resolution>1</resolution>
-            <min_angle>-0.741765</min_angle>
-            <max_angle>0.392699</max_angle>
+            <min_angle>0.0</min_angle>
+            <max_angle>0.0</max_angle>
           </vertical>
         </scan>

File: src/usv_description/urdf/usv.urdf.xacro (robot description, xacro)
@@ -272,11 +272,17 @@
         <parent link="usv_body"/>
         <child link="lidar_front"/>
-        <origin xyz="-0.735 0.885 0.08" rpy="0 0 ${PI/4}"/>
+        <origin xyz="-0.735 0.885 0.50" rpy="0 0 ${PI/4}"/>
     </joint>
     <joint name="lidar_joint_back" type="fixed">
         <parent link="usv_body"/>
         <child link="lidar_back"/>
-        <origin xyz="0.735 -0.885 0.08" rpy="0 0 ${PI/4}"/>
-    </joint>
+        <origin xyz="0.735 -0.885 0.50" rpy="0 0 ${PI/4}"/>
+    </joint>
+    <joint name="usv_body_to_pump" type="fixed">
+         <parent link="usv_body"/>
+        <child link="pump"/>
+        <origin xyz="0 0.630 0.4875" rpy="0 0 0"/>
+    </joint>
+    <!--
     <joint name="usv_body_to_pump" type="prismatic">
          <parent link="usv_body"/>
@@ -290,3 +296,4 @@
             velocity="0.1"/>
     </joint>
+-->
 </robot>
