Commit message: Back up

File: src/usv_description/urdf/usv.urdf.xacro (robot description, xacro)
@@ -272,10 +272,10 @@
         <parent link="usv_body"/>
         <child link="lidar_front"/>
-        <origin xyz="-0.735 0.885 0.50" rpy="0 0 ${PI/4}"/>
+        <origin xyz="-0.735 0.885 0.04" rpy="0 0 ${PI/4}"/>
     </joint>
     <joint name="lidar_joint_back" type="fixed">
         <parent link="usv_body"/>
         <child link="lidar_back"/>
-        <origin xyz="0.735 -0.885 0.50" rpy="0 0 ${PI/4}"/>
+        <origin xyz="0.735 -0.885 0.04" rpy="0 0 ${PI/4}"/>
     </joint>
     <joint name="usv_body_to_pump" type="fixed">
